File: Hardware/Production/MicroMod-RP2040-ProcessorBoard-Panel.brd (EAGLE design)
At the start: 199.6 x 83.1 mm, 790 parts, among them J1 MICROMOD-2222, J10 MICROMOD-2222, J11 MICROMOD-2222, J12 MICROMOD-2222, J13 MICROMOD-2222, J14 MICROMOD-2222, J15 MICROMOD-2222, J16 MICROMOD-2222, J2 MICROMOD-2222, J3 MICROMOD-2222, J4 MICROMOD-2222, J5 MICROMOD-2222, J6 MICROMOD-2222, J7 MICROMOD-2222, J8 MICROMOD-2222, J9 MICROMOD-2222, U1 W25QXX128MBIT, U10 RP2040, U11 W25QXX128MBIT, U12 FSUSB30MUX_MSOP10, U13 RP2040, U14 W25QXX128MBIT, U15 FSUSB30MUX_MSOP10, U16 RP2040, U17 W25QXX128MBIT, U18 FSUSB30MUX_MSOP10, U19 RP2040, U2 FSUSB30MUX_MSOP10, U20 W25QXX128MBIT, U21 FSUSB30MUX_MSOP10, U22 RP2040, U23 W25QXX128MBIT, U24 FSUSB30MUX_MSOP10, U25 RP2040, U26 W25QXX128MBIT, U27 FSUSB30MUX_MSOP10, U28 RP2040, U29 W25QXX128MBIT, U3 RP2040, U30 FSUSB30MUX_MSOP10, U31 RP2040, U32 W25QXX128MBIT, U33 FSUSB30MUX_MSOP10, U34 RP2040, U35 W25QXX128MBIT, U36 FSUSB30MUX_MSOP10, U37 RP2040, U38 W25QXX128MBIT, U39 FSUSB30MUX_MSOP10, U4 RP2040, U40 RP2040, U41 W25QXX128MBIT, U42 FSUSB30MUX_MSOP10, U43 RP2040, U44 W25QXX128MBIT, U45 FSUSB30MUX_MSOP10, U46 RP2040, U47 W25QXX128MBIT, U48 FSUSB30MUX_MSOP10, U5 W25QXX128MBIT, U6 FSUSB30MUX_MSOP10, U7 RP2040, U8 W25QXX128MBIT, U9 FSUSB30MUX_MSOP10, Y1 12MHz, Y10 12MHz, Y11 12MHz, Y12 12MHz, Y13 12MHz, Y14 12MHz, Y15 12MHz, Y16 12MHz, Y2 12MHz, Y3 12MHz, Y4 12MHz, Y5 12MHz, Y6 12MHz, Y7 12MHz, Y8 12MHz, Y9 12MHz

Commit message: Update USB mux prod ID
Parts:
- U2: device RP2040:MSOP10 -> SparkFun-IC-Special-Function:MSOP10

Commit message: Update silk
Parts:
- removed U$113, U$124, U$135, U$146, U$157, U$168: (no value), output:STAT0
- removed U$114, U$118, U$125, U$129, U$136, U$140, U$147, U$151, U$158, U$162, U$169, U$173: (no value), output:PI2
- removed U$115, U$120, U$126, U$131, U$137, U$142, U$148, U$153, U$159, U$164, U$170, U$175: (no value), output:RP20400
- removed U$116, U$121, U$127, U$132, U$138, U$143, U$149, U$154, U$160, U$165, U$171, U$176: (no value), output:_RASPBERRY1
- removed U$117, U$119, U$128, U$130, U$139, U$141, U$150, U$152, U$161, U$163, U$172, U$174: (no value), SparkFun-MicroMod:MICROMOD_LOGO_.3
- removed U$122, U$123, U$133, U$134, U$144, U$145, U$155, U$156, U$166, U$167: (no value), SparkFun-MicroMod:MICROMOD_MI_LOGO_.35
- U$10, U$110, U$33, U$55, U$61, U$83: device output:_RASPBERRY1 -> SparkFun-MicroMod:MICROMOD_LOGO_.3
- U$101, U$24, U$45, U$6: device SparkFun-MicroMod:MICROMOD_MI_LOGO_.35 -> output:STAT0
- U$102, U$14, U$25, U$91: device output:STAT0 -> output:RP20400
- U$103, U$19, U$26, U$41, U$48, U$96: device output:PI2 -> SparkFun-MicroMod:MICROMOD_LOGO_.3
- U$104, U$27, U$54, U$76, U$82: device output:RP20400 -> SparkFun-MicroMod:MICROMOD_LOGO_.3
- U$105, U$28, U$39, U$77, U$88: device output:_RASPBERRY1 -> output:RP20400
- U$106, U$29, U$51, U$64, U$86: device SparkFun-MicroMod:MICROMOD_LOGO_.3 -> SparkFun-MicroMod:MICROMOD_MI_LOGO_.35
- U$107, U$15, U$2, U$30, U$37, U$85, U$92: device output:PI2 -> SparkFun-MicroMod:MICROMOD_MI_LOGO_.35
- U$108, U$31, U$73: device SparkFun-MicroMod:MICROMOD_LOGO_.3 -> output:STAT0
- U$111, U$13, U$34, U$68, U$89, U$90: device SparkFun-MicroMod:MICROMOD_MI_LOGO_.35 -> SparkFun-MicroMod:MICROMOD_LOGO_.3
- U$112, U$35, U$46, U$56, U$67: device SparkFun-MicroMod:MICROMOD_MI_LOGO_.35 -> output:RP20400
- U$16, U$43, U$65, U$71, U$93: device output:RP20400 -> SparkFun-MicroMod:MICROMOD_MI_LOGO_.35
- U$17, U$66, U$94: device output:_RASPBERRY1 -> output:STAT0
- U$18, U$42, U$53, U$84, U$95: device SparkFun-MicroMod:MICROMOD_LOGO_.3 -> output:RP20400
- U$22, U$44, U$5, U$50, U$72, U$99: device output:_RASPBERRY1 -> SparkFun-MicroMod:MICROMOD_MI_LOGO_.35
- U$36, U$58: device output:STAT0 -> SparkFun-MicroMod:MICROMOD_MI_LOGO_.35
- U$38, U$87: device output:RP20400 -> output:STAT0
- U$47, U$69: device output:STAT0 -> SparkFun-MicroMod:MICROMOD_LOGO_.3
- U$52, U$59: device output:PI2 -> output:STAT0
- U$63, U$70, U$74, U$8, U$81: device output:PI2 -> output:RP20400
- U12, U15, U18, U21, U24, U27, U30, U33, U36, U39, U42, U45, U48, U6, U9: device RP2040:MSOP10 -> SparkFun-IC-Special-Function:MSOP10
- moved U$106 153.3 mm to (177.7, 62.9), turned to 90 degrees
- moved U$99 142.1 mm to (155.2, 62.9), flipped to the top, turned to 90 degrees
- moved U$108 139.2 mm to (179.2, 50.2), flipped to the top, turned to 180 degrees
- moved U$61 134.3 mm to (2.82, 57.8)
- moved U$60 134.2 mm to (4.47, 57.9)
- moved U$94 128.5 mm to (134.2, 50.2), turned to 180 degrees
- moved U$92 127.2 mm to (132.7, 62.9), turned to 90 degrees
- moved U$62 127.0 mm to (16.3, 63.1), flipped to the bottom, turned to 270 degrees
- moved U$104 124.9 mm to (151.3, 63.1), flipped to the bottom
- moved U$110 124.9 mm to (160.4, 57.8), flipped to the top, turned to 90 degrees
- moved U$105 124.7 mm to (153.1, 63.0), flipped to the bottom
- moved U$109 123.3 mm to (162.0, 57.9), flipped to the top, turned to 90 degrees
- moved U$107 122.8 mm to (159.8, 53.9)
- moved U$67 121.3 mm to (27.0, 57.9)
- moved U$68 120.8 mm to (25.3, 57.8), flipped to the top, turned to 90 degrees
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